Commit message: add mobile dual arm with sucker

File: mobile_dual_arm_description/urdf/mobile_dual_arm.ros2_control.xacro (robot description, xacro)
@@ -57,5 +57,5 @@
         <state_interface name="effort"/>
       </joint>
-      <!-- <joint name="r_joint_7">
+      <joint name="r_joint_7">
         <param name="id">7</param>
         <command_interface name="position"/>
@@ -64,5 +64,5 @@
         <state_interface name="velocity"/>
         <state_interface name="effort"/>
-      </joint> -->
+      </joint>
       <joint name="l_joint_1">
         <param name="id">1</param>
@@ -113,64 +113,13 @@
         <state_interface name="effort"/>
       </joint>
-    </ros2_control>
-  <!-- <ros2_control name="GazeboSystem" type="system">
-    <hardware>
-      <plugin>gazebo_ros2_control/GazeboSystem</plugin>
-    </hardware>
-      <joint name="${side}_tool_joint">
+      <joint name="l_joint_7">
+        <param name="id">7</param>
         <command_interface name="position"/>
         <command_interface name="velocity"/>
-        <param name="min">-1</param>
-        <param name="max">1</param>
         <state_interface name="position"/>
         <state_interface name="velocity"/>
         <state_interface name="effort"/>
       </joint>
-      <joint name="${side}_end_joint1">
-        <command_interface name="position"/>
-        <command_interface name="velocity"/>
-        <param name="min">-1</param>
-        <param name="max">1</param>
-        <state_interface name="position"/>
-        <state_interface name="velocity"/>
-        <state_interface name="effort"/>
-      </joint>
-      <joint name="${side}_end_joint2">
-        <command_interface name="position"/>
-        <command_interface name="velocity"/>
-        <param name="min">-1</param>
-        <param name="max">1</param>
-        <state_interface name="position"/>
-        <state_interface name="velocity"/>
-        <state_interface name="effort"/>
-      </joint>
-      <joint name="${side}_end_joint3">
-        <command_interface name="position"/>
-        <command_interface name="velocity"/>
-        <param name="min">-1</param>
-        <param name="max">1</param>
-        <state_interface name="position"/>
-        <state_interface name="velocity"/>
-        <state_interface name="effort"/>
-      </joint>
-      <joint name="${side}_end_joint4">
-        <command_interface name="position"/>
-        <command_interface name="velocity"/>
-        <param name="min">-1</param>
-        <param name="max">1</param>
-        <state_interface name="position"/>
-        <state_interface name="velocity"/>
-        <state_interface name="effort"/>
-      </joint>
-      <joint name="${side}_end_joint5">
-        <command_interface name="position"/>
-        <command_interface name="velocity"/>
-        <param name="min">-1</param>
-        <param name="max">1</param>
-        <state_interface name="position"/>
-        <state_interface name="velocity"/>
-        <state_interface name="effort"/>
-      </joint>
-  </ros2_control> -->
+    </ros2_control>
   </xacro:macro>
 </robot>

File: mobile_dual_arm_description/urdf/mobile_dual_arm_sucker.xacro (robot description, xacro)
@@ -7,5 +7,5 @@
   <xacro:include filename="$(find timda_body)/urdf/timda_body.xacro" />
   <!-- <xacro:include filename="$(find slide_rail)/urdf/slide_rail.xacro" /> -->
-  <!-- <xacro:include filename="$(find suction_urdf)/urdf/suction_urdf.xacro" /> -->
+  <xacro:include filename="$(find suction_urdf)/urdf/suction_urdf.xacro" />
   <!-- <xacro:include filename="$(find single_arm_description)/urdf/materials.xacro" /> -->
   <!-- <xacro:include filename="$(find mobile_dual_arm_description)/urdf/mobile_dual_arm.gazebo" /> -->
@@ -14,4 +14,5 @@
   <xacro:include filename="$(find mir_description)/urdf/mir.ros2_control.xacro" />
   <xacro:include filename="$(find timda_body)/urdf/timda_body.ros2_control.xacro" />
+  <xacro:include filename="$(find suction_urdf)/urdf/suction.ros2_control.xacro" />
   <link name="world"/>
     <!-- <link name="world"/>
@@ -49,26 +50,16 @@
   </joint>
   <xacro:mir_100 prefix="mobile_" ns=""/>
-  <link name="r_tool_link">
-    <visual>
-      <origin xyz="0 0 0" rpy="0 0 0"/>
-      <geometry>
-        <box size="0.001 0.001 0.001"/>
-      </geometry>
-    </visual>
-  </link>
-  <link name="l_tool_link">
-    <visual>
-      <origin xyz="0 0 0" rpy="0 0 0"/>
-      <geometry>
-        <box size="0.001 0.001 0.001"/>
-      </geometry>
-    </visual>
-  </link>
   <xacro:single_arm side="r_"  parent="slide_right" child="r_tool_link" toolrot="-1.57">
     <origin xyz="0.0 0.1151 0.0" rpy="1.57 3.1415926 3.1415926" />
   </xacro:single_arm>
+  <xacro:suction side="r"  parent="r_tool_link">
+    <origin xyz="0 -0.016 0" rpy="0 0 -1.57" />
+  </xacro:suction>
   <xacro:single_arm side="l_"  parent="slide_left" child="l_tool_link" toolrot="1.57">
     <origin xyz="0.0 0.1151 0.0" rpy="-1.57 0 0" />
   </xacro:single_arm>
+  <xacro:suction side="l"  parent="l_tool_link">
+    <origin xyz="0 0.016 0" rpy="0 0 1.57" />
+  </xacro:suction>
   <!--joint name="fixed" type="fixed">
     <origin
@@ -140,8 +131,9 @@
     <child link="Bin"/>
   </joint>
-  <!-- <xacro:mobile_dual_arm_ros2_control name="mobile_dual_arm_ros2_control"/> -->
   <xacro:single_arm_ros2_control name="right_single_arm_ros2_control" side="r_"/>
   <xacro:single_arm_ros2_control name="left_single_arm_ros2_control" side="l_"/>
   <xacro:mir_100_ros2_control prefix = "mobile_" name ="mir_100_ros2_control" />
   <xacro:timda_body_ros2_control name ="timda_body_ros2_control" />
+  <xacro:suction_ros2_control name="right_suction_ros2_control" side="r_"/>
+  <xacro:suction_ros2_control name="left_suction_ros2_control" side="l_"/>
 </robot>

File: single_arm_description/urdf/single_arm.ros2_control.xacro (robot description, xacro)
@@ -57,4 +57,12 @@
         <state_interface name="effort"/>
       </joint>
+      <joint name="${side}joint_7">
+        <param name="id">7</param>
+        <command_interface name="position"/>
+        <command_interface name="velocity"/>
+        <state_interface name="position"/>
+        <state_interface name="velocity"/>
+        <state_interface name="effort"/>
+      </joint>
     </ros2_control>
   </xacro:macro>

File: single_arm_description/urdf/single_arm.urdf.xacro (robot description, xacro)
@@ -4,11 +4,19 @@
   <xacro:include filename="$(find single_arm_description)/urdf/single_arm.ros2_control.xacro" />
   <link name="world"/>
-  <xacro:single_arm parent="world" side="" child="" toolrot="-1.57">
+  <!-- <xacro:single_arm parent="world" side="" child="" toolrot="-1.57">
+    <origin xyz="0 0 0.1" rpy="0 0 0" />
+  </xacro:single_arm> -->
+  <!-- <link name="r_tool_link"/> -->
+  <link name="tool_link">
+    <visual>
+      <origin xyz="0 0 0" rpy="0 0 0"/>
+      <geometry>
+        <box size="0.001 0.001 0.001"/>
+      </geometry>
+    </visual>
+  </link>
+  <xacro:single_arm side=""  parent="world" child="tool_link" toolrot="-1.57">
     <origin xyz="0 0 0.1" rpy="0 0 0" />
   </xacro:single_arm>
-  <!-- <link name="r_tool_link"/> -->
-  <!-- <xacro:single_arm side="r"  parent="slide_right" child="r_tool_link" toolrot="-1.57">
-    <origin xyz="0.0 0.1151 0.0" rpy="1.57 3.1415926 3.1415926" />
-  </xacro:single_arm> -->
   <xacro:single_arm_ros2_control name="single_arm_ros2_control" side=""/>
 </robot>

File: single_arm_description/urdf/single_arm.xacro (robot description, xacro)
@@ -430,6 +430,5 @@
 	    </collision>
 	  </link> -->
-<!--
-      <xacro:if value="${(side == 'r_') or (side == 'l_')}">
+      <!-- <xacro:if value="${'link' in child}">
 		<joint
 			name="${side}joint_7"
@@ -455,14 +454,14 @@
 		</joint>
     </xacro:if> -->
-		<!-- <joint
+		<joint
 			name="${side}joint_7"
 			type="revolute">
 			<origin
 				xyz="0 0.03680 0.135"
-				rpy="0 0 ${toolrot}" /> -->
+				rpy="0 0 ${toolrot}" />
 				<!-- rpy="1.5708 ${toolrot} 0" /> -->
 				<!-- xyz="-0.008041 0.038 0.13545" -->
 				<!-- xyz="-0.0025 0.038 0.135" -->
-			<!-- <parent
+			<parent
 				link="${side}link_6" />
 			<child
@@ -476,5 +475,5 @@
                 velocity="6.5" />
           <dynamics damping="0.7"/>
-		</joint> -->
+		</joint>
           <!--
 	  <link
