Commit message: add use fake hardware with mobile dual arm, heading on slider hardware interface

File: mobile_dual_arm_description/urdf/mobile_dual_arm.xacro (robot description, xacro)
@@ -140,8 +140,8 @@
     <child link="Bin"/>
   </joint>
-  <!-- <xacro:mobile_dual_arm_ros2_control name="mobile_dual_arm_ros2_control"/> -->
-  <xacro:single_arm_ros2_control name="right_single_arm_ros2_control" side="r_"/>
-  <xacro:single_arm_ros2_control name="left_single_arm_ros2_control" side="l_"/>
+  <xacro:arg name="use_fake_hardware" default="true" />
+  <xacro:single_arm_ros2_control name="right_single_arm_ros2_control" side="r_" use_fake_hardware="$(arg use_fake_hardware)"/>
+  <xacro:single_arm_ros2_control name="left_single_arm_ros2_control" side="l_" use_fake_hardware="$(arg use_fake_hardware)"/>
   <xacro:mir_100_ros2_control prefix = "mobile_" name ="mir_100_ros2_control" />
-  <xacro:timda_body_ros2_control name ="timda_body_ros2_control" />
+  <xacro:timda_body_ros2_control name ="timda_body_ros2_control" use_fake_hardware="$(arg use_fake_hardware)"/>
 </robot>

File: mobile_dual_arm_description/urdf/mobile_dual_arm_sucker.xacro (robot description, xacro)
@@ -131,8 +131,9 @@
     <child link="Bin"/>
   </joint>
-  <xacro:single_arm_ros2_control name="right_single_arm_ros2_control" side="r_"/>
-  <xacro:single_arm_ros2_control name="left_single_arm_ros2_control" side="l_"/>
+  <xacro:arg name="use_fake_hardware" default="true" />
+  <xacro:single_arm_ros2_control name="right_single_arm_ros2_control" side="r_" use_fake_hardware="$(arg use_fake_hardware)"/>
+  <xacro:single_arm_ros2_control name="left_single_arm_ros2_control" side="l_" use_fake_hardware="$(arg use_fake_hardware)"/>
   <xacro:mir_100_ros2_control prefix = "mobile_" name ="mir_100_ros2_control" />
-  <xacro:timda_body_ros2_control name ="timda_body_ros2_control" />
+  <xacro:timda_body_ros2_control name ="timda_body_ros2_control" use_fake_hardware="$(arg use_fake_hardware)"/>
   <xacro:suction_ros2_control name="right_suction_ros2_control" side="r_"/>
   <xacro:suction_ros2_control name="left_suction_ros2_control" side="l_"/>

File: single_arm_description/urdf/single_arm.ros2_control.xacro (robot description, xacro)
@@ -1,5 +1,5 @@
 <?xml version="1.0"?>
 <robot xmlns:xacro="http://www.ros.org/wiki/xacro">
-  <xacro:macro name="single_arm_ros2_control" params="name side">
+  <xacro:macro name="single_arm_ros2_control" params="name side use_fake_hardware=true">
     <ros2_control name="${name}" type="system">
       <hardware>
@@ -7,5 +7,7 @@
         <param name="usb_port">/dev/ttyUSB0</param>
         <param name="baud_rate">115200</param>
-        <param name="use_dummy">true</param>
+        <xacro:if value="${use_fake_hardware}">
+          <param name="use_dummy">true</param>
+        </xacro:if>
       </hardware>
       <joint name="${side}joint_1">

Commit message: add usb port with mobile dual arm, heading on slider hardware interface

File: mobile_dual_arm_description/urdf/mobile_dual_arm.xacro (robot description, xacro)
@@ -141,7 +141,11 @@
   </joint>
   <xacro:arg name="use_fake_hardware" default="true" />
-  <xacro:single_arm_ros2_control name="right_single_arm_ros2_control" side="r_" use_fake_hardware="$(arg use_fake_hardware)"/>
-  <xacro:single_arm_ros2_control name="left_single_arm_ros2_control" side="l_" use_fake_hardware="$(arg use_fake_hardware)"/>
+  <xacro:arg name="right_arm_port" default="wrs/arm_right" />
+  <xacro:arg name="left_arm_port" default="wrs/arm_left" />
+  <xacro:single_arm_ros2_control name = "right_single_arm_ros2_control" side = "r_" use_fake_hardware = "$(arg use_fake_hardware)" usb_port = "$(arg right_arm_port)"/>
+  <xacro:single_arm_ros2_control name = "left_single_arm_ros2_control" side = "l_" use_fake_hardware = "$(arg use_fake_hardware)" usb_port = "$(arg left_arm_port)"/>
   <xacro:mir_100_ros2_control prefix = "mobile_" name ="mir_100_ros2_control" />
-  <xacro:timda_body_ros2_control name ="timda_body_ros2_control" use_fake_hardware="$(arg use_fake_hardware)"/>
+  <xacro:timda_body_ros2_control name ="timda_body_ros2_control"  side = "right" use_fake_hardware="$(arg use_fake_hardware)"/>
+  <xacro:timda_body_ros2_control name ="right_slider_ros2_control"  side = "right" use_fake_hardware="$(arg use_fake_hardware)"/>
+  <xacro:timda_body_ros2_control name ="left_slider_ros2_control" side = "left" use_fake_hardware="$(arg use_fake_hardware)"/>
 </robot>

File: mobile_dual_arm_description/urdf/mobile_dual_arm_sucker.xacro (robot description, xacro)
@@ -132,9 +132,12 @@
   </joint>
   <xacro:arg name="use_fake_hardware" default="true" />
-  <xacro:single_arm_ros2_control name="right_single_arm_ros2_control" side="r_" use_fake_hardware="$(arg use_fake_hardware)"/>
-  <xacro:single_arm_ros2_control name="left_single_arm_ros2_control" side="l_" use_fake_hardware="$(arg use_fake_hardware)"/>
+  <xacro:arg name="right_arm_port" default="wrs/arm_right" />
+  <xacro:arg name="left_arm_port" default="wrs/arm_left" />
+  <xacro:single_arm_ros2_control name = "right_single_arm_ros2_control" side = "r_" use_fake_hardware = "$(arg use_fake_hardware)" usb_port = "$(arg right_arm_port)"/>
+  <xacro:single_arm_ros2_control name = "left_single_arm_ros2_control" side = "l_" use_fake_hardware = "$(arg use_fake_hardware)" usb_port = "$(arg left_arm_port)"/>
   <xacro:mir_100_ros2_control prefix = "mobile_" name ="mir_100_ros2_control" />
-  <xacro:timda_body_ros2_control name ="timda_body_ros2_control" use_fake_hardware="$(arg use_fake_hardware)"/>
-  <xacro:suction_ros2_control name="right_suction_ros2_control" side="r_"/>
-  <xacro:suction_ros2_control name="left_suction_ros2_control" side="l_"/>
+  <xacro:timda_body_ros2_control name ="right_slider_ros2_control"  side = "right" use_fake_hardware="$(arg use_fake_hardware)"/>
+  <xacro:timda_body_ros2_control name ="left_slider_ros2_control" side = "left" use_fake_hardware="$(arg use_fake_hardware)"/>
+  <xacro:suction_ros2_control name = "right_suction_ros2_control" side = "r_"/>
+  <xacro:suction_ros2_control name = "left_suction_ros2_control" side = "l_"/>
 </robot>

File: single_arm_description/urdf/single_arm.ros2_control.xacro (robot description, xacro)
@@ -1,9 +1,13 @@
 <?xml version="1.0"?>
 <robot xmlns:xacro="http://www.ros.org/wiki/xacro">
-  <xacro:macro name="single_arm_ros2_control" params="name side use_fake_hardware=true">
+  <xacro:macro name="single_arm_ros2_control" params="
+    name
+    side
+    usb_port:=/dev/ttyUSB0
+    use_fake_hardware:=true">
     <ros2_control name="${name}" type="system">
       <hardware>
         <plugin>dynamixel_hardware/DynamixelHardware</plugin>
-        <param name="usb_port">/dev/ttyUSB0</param>
+        <param name="usb_port">${usb_port}</param>
         <param name="baud_rate">115200</param>
         <xacro:if value="${use_fake_hardware}">

File: timda_body/urdf/timda_body.ros2_control.xacro (robot description, xacro)
@@ -3,4 +3,5 @@
   <xacro:macro name="timda_body_ros2_control" params="
     name
+    side
     use_fake_hardware:=true fake_sensor_commands:=true
     sim_gazebo:=false
@@ -28,13 +29,5 @@
       </hardware>
 <!-- <command_interface name="velocity"/> -->
-      <joint name="joint_right">
-        <command_interface name="position"/>
-        <param name="min">-1</param>
-        <param name="max">1</param>
-        <state_interface name="position"/>
-        <state_interface name="velocity"/>
-        <state_interface name="effort"/>
-      </joint>
-      <joint name="joint_left">
+      <joint name="joint_${side}">
         <command_interface name="position"/>
         <param name="min">-1</param>

Commit message: fixing slider hardware, heading to test

File: mobile_dual_arm_description/urdf/mobile_dual_arm.xacro (robot description, xacro)
@@ -143,6 +143,6 @@
   <xacro:arg name="right_arm_port" default="/dev/wrs/arm_right" />
   <xacro:arg name="left_arm_port" default="/dev/wrs/arm_left" />
-  <xacro:single_arm_ros2_control name = "right_single_arm_ros2_control" side = "r_" use_fake_hardware = "$(arg use_fake_hardware)" usb_port = "$(arg right_arm_port)"/>
-  <xacro:single_arm_ros2_control name = "left_single_arm_ros2_control" side = "l_" use_fake_hardware = "$(arg use_fake_hardware)" usb_port = "$(arg left_arm_port)"/>
+  <xacro:single_arm_ros2_control name = "right_single_arm_ros2_control" side = "r_" use_fake_hardware = "true" usb_port = "$(arg right_arm_port)"/>
+  <xacro:single_arm_ros2_control name = "left_single_arm_ros2_control" side = "l_" use_fake_hardware = "true" usb_port = "$(arg left_arm_port)"/>
   <xacro:mir_100_ros2_control prefix = "mobile_" name ="mir_100_ros2_control" />
   <xacro:timda_body_ros2_control name ="right_slider_ros2_control"  side = "right" use_fake_hardware="$(arg use_fake_hardware)"/>

File: mobile_dual_arm_description/urdf/mobile_dual_arm_sucker.xacro (robot description, xacro)
@@ -83,5 +83,5 @@
     <child link="Arm_Base_R"/>
   </joint-->
-  <link name="Bin">
+  <!-- <link name="Bin">
     <inertial>
       <origin
@@ -130,6 +130,7 @@
     <parent link="base_link"/>
     <child link="Bin"/>
-  </joint>
+  </joint> -->
   <xacro:arg name="use_fake_hardware" default="true" />
+  <xacro:arg name="use_real_hardware" default="false" />
   <xacro:arg name="right_arm_port" default="/dev/wrs/arm_right" />
   <xacro:arg name="left_arm_port" default="/dev/wrs/arm_left" />
@@ -137,6 +138,6 @@
   <xacro:single_arm_ros2_control name = "left_single_arm_ros2_control" side = "l_" use_fake_hardware = "$(arg use_fake_hardware)" usb_port = "$(arg left_arm_port)"/>
   <xacro:mir_100_ros2_control prefix = "mobile_" name ="mir_100_ros2_control" />
-  <xacro:timda_body_ros2_control name ="right_slider_ros2_control"  side = "right" use_fake_hardware="$(arg use_fake_hardware)"/>
-  <xacro:timda_body_ros2_control name ="left_slider_ros2_control" side = "left" use_fake_hardware="$(arg use_fake_hardware)"/>
+  <xacro:timda_body_ros2_control name ="right_slider_ros2_control"  side = "right" use_fake_hardware="$(arg use_real_hardware)"/>
+  <xacro:timda_body_ros2_control name ="left_slider_ros2_control" side = "left" use_fake_hardware="$(arg use_real_hardware)"/>
   <xacro:suction_ros2_control name = "right_suction_ros2_control" side = "r_"/>
   <xacro:suction_ros2_control name = "left_suction_ros2_control" side = "l_"/>
